File: Emmelie-v3.2.brd (EAGLE design)
At the start: 188 x 124 mm, 57 parts, among them IC10 TL072P, IC11 TL072P, IC12 TL072P, IC13 TL072P, IC14 TL072P, IC9 TL072P, J2 22-27-2041-04, J3 22-27-2041-04

Commit message: tidied up a little in schematic and board
Parts:
- added U$13: (no value), frames:A4L-LOC
Changed lines of the file:
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@@
 <layer number="46" name="Milling" color="3" fill="1" visible="no" active="yes"/>
 <layer number="47" name="Measures" color="7" fill="1" visible="no" active="yes"/>
-<layer number="48" name="Document" color="7" fill="1" visible="no" active="yes"/>
+<layer number="48" name="Document" color="7" fill="1" visible="yes" active="yes"/>
 <layer number="49" name="Reference" color="7" fill="1" visible="no" active="yes"/>
 <layer number="50" name="dxf" color="7" fill="1" visible="yes" active="yes"/>
 <layer number="51" name="tDocu" color="7" fill="1" visible="yes" active="yes"/>
 <layer number="52" name="bDocu" color="7" fill="1" visible="no" active="yes"/>
+<layer number="90" name="Modules" color="5" fill="1" visible="no" active="no"/>
 <layer number="91" name="Nets" color="2" fill="1" visible="no" active="no"/>
 <layer number="92" name="Busses" color="1" fill="1" visible="no" active="no"/>
@@
 <element name="U$11" library="Mario - Klinke Stecker 3,5" package="KLINKE3,5" value="KLINKE3,5" x="92" y="36" smashed="yes"/>
 <element name="U$12" library="Mario - Klinke Stecker 3,5" package="KLINKE3,5" value="KLINKE3,5" x="104" y="36" smashed="yes"/>
+<element name="U$13" library="frames" library_urn="urn:adsk.eagle:library:229" package="A4L-LOC" value="" x="-36" y="-120" smashed="yes">
+<attribute name="DRAWING_NAME" x="181.17" y="-104.76" size="2.54" layer="48" font="vector"/>
+<attribute name="LAST_DATE_TIME" x="181.17" y="-109.84" size="2.286" layer="48" font="vector"/>
+</element>
 </elements>
 <signals>
@@
 </board>
 </drawing>
+<compatibility>
+<note version="8.2" severity="warning">
+Since Version 8.2, EAGLE supports online libraries. The ids
+of those online libraries will not be understood (or retained)
+with this version.
+</note>
+<note version="8.3" severity="warning">
+Since Version 8.3, EAGLE supports URNs for individual library
+assets (packages, symbols, and devices). The URNs of those assets
+will not be understood (or retained) with this version.
+</note>
+</compatibility>
 </eagle>
