File: Emmelie-v3.2.sch (EAGLE design)
At the start: 57 parts, among them IC10 TL072P, IC11 TL072P, IC12 TL072P, IC13 TL072P, IC14 TL072P, IC9 TL072P, J2 22-27-2041-04, J3 22-27-2041-04

Commit message: tidied up a little in schematic and board
Other:
- note added: "Amplifier + Power supply"
- note added: "Music in/out"
- note added: "Switches"
