File: AB-AudioMatrix-6x6.sch (EAGLE design)
At the start: 52 parts, among them IC10 TL072D, IC11 TL072D, IC12 TL072D, IC13 TL072D, IC14 TL072D, IC9 TL072D

Commit message: Platine grundlegend fertiggestellt
Parts:
- U$1: MF (none) -> Switchcraft; MFN (none) -> 35RAPC4BH3; MOUSER (none) -> 502-35RAPC4BH3; RS-ONLINE (none) -> 878-7229
Other:
- note added: "FFC Connector IN"
- note added: "FFC Connector OUT"
- note added: "Music IN"
- note added: "Music OUT"
- note added: "Power supply for buffer amplifier"
- note added: "Switches + Buffer amplifier"
- note removed: "Music in/out"
- note removed: "Switches"
- moved on the sheet: IC10A, IC10B, IC11A, IC11B, IC12A, IC12B, IC13A, IC13B, IC14A, IC14B, IC9A, IC9B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

Commit message: 3,5 mm Klinken Buchsen ausgetauscht | Spannungsversorgung hinzugefügt | Fusion 3D-Modell vollständig
Parts:
- removed U$1, U$10, U$11, U$12, U$2, U$3, U$4, U$5, U$6, U$7, U$8, U$9: KLINKE3,5, Mario - Klinke Stecker 3,5:KLINKE3,5
- added J8: (no value), Wurth_Connectors_WR-TBL Wire Protector:691102710003
- added X1, X10, X11, X12, X2, X3, X4, X5, X6, X7, X8, X9: 35RAPC4BH3-2, h8-conector:35RAPC4BH3-2
Connections:
- net +12V: now also J8.1
- net -12V: now also J8.3
- net GND: now also J8.2, X1.GND, X1.LEFT_OFF, X1.RIGHT_OFF, X10.GND, X10.LEFT_OFF, X10.RIGHT_OFF, X11.GND, X11.LEFT_OFF, X11.RIGHT_OFF, X12.GND, X12.LEFT_OFF, X12.RIGHT_OFF, X2.GND, X2.LEFT_OFF, X2.RIGHT_OFF, X3.GND, X3.LEFT_OFF, X3.RIGHT_OFF, X4.GND, X4.LEFT_OFF, X4.RIGHT_OFF, X5.GND, X5.LEFT_OFF, X5.RIGHT_OFF, X6.GND, X6.LEFT_OFF, X6.RIGHT_OFF, X7.GND, X7.LEFT_OFF, X7.RIGHT_OFF, X8.GND, X8.LEFT_OFF, X8.RIGHT_OFF, X9.GND, X9.LEFT_OFF, X9.RIGHT_OFF; no longer U$1.GND, U$1.LEFT_OFF, U$1.RIGHT_OFF, U$10.GND, U$10.LEFT_OFF, U$10.RIGHT_OFF, U$11.GND, U$11.LEFT_OFF, U$11.RIGHT_OFF, U$12.GND, U$12.LEFT_OFF, U$12.RIGHT_OFF, U$2.GND, U$2.LEFT_OFF, U$2.RIGHT_OFF, U$3.GND, U$3.LEFT_OFF, U$3.RIGHT_OFF, U$4.GND, U$4.LEFT_OFF, U$4.RIGHT_OFF, U$5.GND, U$5.LEFT_OFF, U$5.RIGHT_OFF, U$6.GND, U$6.LEFT_OFF, U$6.RIGHT_OFF, U$7.GND, U$7.LEFT_OFF, U$7.RIGHT_OFF, U$8.GND, U$8.LEFT_OFF, U$8.RIGHT_OFF, U$9.GND, U$9.LEFT_OFF, U$9.RIGHT_OFF
- net IN1L: now also X1.LEFT; no longer U$1.LEFT
- net IN1R: now also X1.RIGHT; no longer U$1.RIGHT
- net IN2L: now also X2.LEFT; no longer U$2.LEFT
- net IN2R: now also X2.RIGHT; no longer U$2.RIGHT
- net IN3L: now also X3.LEFT; no longer U$3.LEFT
- net IN3R: now also X3.RIGHT; no longer U$3.RIGHT
- net IN4L: now also X4.LEFT; no longer U$4.LEFT
- net IN4R: now also X4.RIGHT; no longer U$4.RIGHT
- net IN5L: now also X5.LEFT; no longer U$5.LEFT
- net IN5R: now also X5.RIGHT; no longer U$5.RIGHT
- net IN6L: now also X6.LEFT; no longer U$6.LEFT
- net IN6R: now also X6.RIGHT; no longer U$6.RIGHT
- net OUT1L: now also X7.LEFT; no longer U$7.LEFT
- net OUT1R: now also X7.RIGHT; no longer U$7.RIGHT
- net OUT2L: now also X8.LEFT; no longer U$8.LEFT
- net OUT2R: now also X8.RIGHT; no longer U$8.RIGHT
- net OUT3L: now also X9.LEFT; no longer U$9.LEFT
- net OUT3R: now also X9.RIGHT; no longer U$9.RIGHT
- net OUT4L: now also X10.LEFT; no longer U$10.LEFT
- net OUT4R: now also X10.RIGHT; no longer U$10.RIGHT
- net OUT5L: now also X11.LEFT; no longer U$11.LEFT
- net OUT5R: now also X11.RIGHT; no longer U$11.RIGHT
- net OUT6L: now also X12.LEFT; no longer U$12.LEFT
- net OUT6R: now also X12.RIGHT; no longer U$12.RIGHT
Other:
- note added: "Symmetrical Power Supply"
- note added: "Symmetrical power supply is allowd to have a range from ±5 to ±30 VDC"
- moved on the sheet: R13, R14, R15, R16, R17, R18, R19, R20, R21, R22, R23, R24
